File: 2022/LocoMainBoard/Capacitor Management.kicad_sch (KiCad schematic)
At the start: 105 parts, among them J28 Screw Terminal, J29 Screw Terminal, J30 Screw Terminal, J31 Mini-Fit Jr 2x01, Q19 Q_NMOS_SSSGD, Q20 Q_NMOS_SSSGD, Q21 Q_NMOS_SSSGD, Q22 Q_NMOS_SSSGD, Q23 Q_NMOS_SSSGD, Q24 Q_NMOS_SSSGD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

Commit message: Full Rework of PCB --> basically V2
Connections:
- net +VBAT: no longer C105.1, D26.2 (A), D27.2 (A), Q20.5 (D)
- new net +VBAT_B: C105.1, D26.2 (A), D27.2 (A), Q20.5 (D)
Changed lines of the file:
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@@
     (pin "2")
-  )
-  (symbol (lib_id "RCAS_Power_Symbols:+VBAT_Enabled") (at 173.99 80.01 0) (unit 1)
-    (in_bom yes) (on_board yes)
-    (property "Reference" "#PWR0231" (id 0) (at 173.99 83.82 0)
-      (effects (font (size 1.27 1.27)) hide)
-    )
-    (property "Value" "+VBAT_Enabled" (id 1) (at 174.371 75.6158 0))
-    (property "Footprint" "" (id 2) (at 173.99 80.01 0)
-      (effects (font (size 1.27 1.27)) hide)
-    )
-    (property "Datasheet" "" (id 3) (at 173.99 80.01 0)
-      (effects (font (size 1.27 1.27)) hide)
-    )
-    (pin "1")
-  )
-  (symbol (lib_id "RCAS_Power_Symbols:+VBAT_Enabled") (at 156.21 113.03 0) (unit 1)
-    (in_bom yes) (on_board yes)
-    (property "Reference" "#PWR0230" (id 0) (at 156.21 116.84 0)
-      (effects (font (size 1.27 1.27)) hide)
-    )
-    (property "Value" "+VBAT_Enabled" (id 1) (at 156.591 108.6358 0))
-    (property "Footprint" "" (id 2) (at 156.21 113.03 0)
-      (effects (font (size 1.27 1.27)) hide)
-    )
-    (property "Datasheet" "" (id 3) (at 156.21 113.03 0)
-      (effects (font (size 1.27 1.27)) hide)
-    )
-    (pin "1")
-  )
-  (symbol (lib_id "RCAS_Power_Symbols:+VBAT_Enabled") (at 129.54 121.92 0) (unit 1)
-    (in_bom yes) (on_board yes)
-    (property "Reference" "#PWR0229" (id 0) (at 129.54 125.73 0)
-      (effects (font (size 1.27 1.27)) hide)
-    )
-    (property "Value" "+VBAT_Enabled" (id 1) (at 129.921 117.5258 0))
-    (property "Footprint" "" (id 2) (at 129.54 121.92 0)
-      (effects (font (size 1.27 1.27)) hide)
-    )
-    (property "Datasheet" "" (id 3) (at 129.54 121.92 0)
-      (effects (font (size 1.27 1.27)) hide)
-    )
-    (pin "1")
   )
   (symbol (lib_id "RCAS_Test_Points:TestPoint") (at 135.89 151.13 180) (unit 1)
@@
       (effects (font (size 1.27 1.27)) hide)
     )
+    (pin "1")
+  )
+  (symbol (lib_id "RCAS_Power_Symbols:+VBAT_B") (at 156.21 113.03 0) (unit 1)
+    (in_bom yes) (on_board yes) (fields_autoplaced)
+    (property "Reference" "#PWR?" (id 0) (at 156.21 116.84 0)
+      (effects (font (size 1.27 1.27)) hide)
+    )
+    (property "Value" "+VBAT_B" (id 1) (at 156.21 109.4542 0))
+    (property "Footprint" "" (id 2) (at 156.21 113.03 0)
+      (effects (font (size 1.27 1.27)) hide)
+    )
+    (property "Datasheet" "" (id 3) (at 156.21 113.03 0)
+      (effects (font (size 1.27 1.27)) hide)
+    )
+    (pin "1")
+  )
+  (symbol (lib_id "RCAS_Power_Symbols:+VBAT_B") (at 129.54 121.92 0) (unit 1)
+    (in_bom yes) (on_board yes) (fields_autoplaced)
+    (property "Reference" "#PWR?" (id 0) (at 129.54 125.73 0)
+      (effects (font (size 1.27 1.27)) hide)
+    )
+    (property "Value" "+VBAT_B" (id 1) (at 129.54 118.3442 0))
+    (property "Footprint" "" (id 2) (at 129.54 121.92 0)
+      (effects (font (size 1.27 1.27)) hide)
+    )
+    (property "Datasheet" "" (id 3) (at 129.54 121.92 0)
+      (effects (font (size 1.27 1.27)) hide)
+    )
+    (pin "1")
+  )
+  (symbol (lib_id "RCAS_Power_Symbols:+VBAT_B") (at 173.99 80.01 0) (unit 1)
+    (in_bom yes) (on_board yes) (fields_autoplaced)
+    (property "Reference" "#PWR?" (id 0) (at 173.99 83.82 0)
+      (effects (font (size 1.27 1.27)) hide)
+    )
+    (property "Value" "+VBAT_B" (id 1) (at 173.99 76.4342 0))
+    (property "Footprint" "" (id 2) (at 173.99 80.01 0)
+      (effects (font (size 1.27 1.27)) hide)
+    )
+    (property "Datasheet" "" (id 3) (at 173.99 80.01 0)
+      (effects (font (size 1.27 1.27)) hide)
+    )
