File: 2022/LocoMainBoard/Isolated Monitoring.kicad_sch (KiCad schematic)
At the start: 36 parts, among them J11 Mini-Fit Jr 2x01, J12 Mini-Fit Jr 2x01, J13 Mini-Fit Jr 2x02, U13 TLV70220PDBVR, U14 MCP3424

Commit message: Full Rework of PCB --> basically V2
Connections:
- net +VBAT renamed +VBAT_B
Changed lines of the file:
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@@
     (pin "2")
   )
-  (symbol (lib_id "RCAS_Power_Symbols:+VBAT_Enabled") (at 207.01 81.28 0) (unit 1)
-    (in_bom yes) (on_board yes)
-    (property "Reference" "#PWR095" (id 0) (at 207.01 85.09 0)
+  (symbol (lib_id "RCAS_Power_Symbols:+VBAT_B") (at 207.01 81.28 0) (unit 1)
+    (in_bom yes) (on_board yes) (fields_autoplaced)
+    (property "Reference" "#PWR?" (id 0) (at 207.01 85.09 0)
       (effects (font (size 1.27 1.27)) hide)
     )
-    (property "Value" "+VBAT_Enabled" (id 1) (at 207.391 76.8858 0))
+    (property "Value" "+VBAT_B" (id 1) (at 207.01 77.7042 0))
     (property "Footprint" "" (id 2) (at 207.01 81.28 0)
       (effects (font (size 1.27 1.27)) hide)
