File: 2022/LocoMainBoard/Isolated Power.kicad_sch (KiCad schematic)
At the start: 21 parts, among them J8 Mini-Fit Jr 2x01, Q12 2N7002, U10 LMR16006

Commit message: Full Rework of PCB --> basically V2
Connections:
- net +VBAT: no longer C26.1, C27.1, R40.1, R41.1, R42.1, U10.5 (VIN)
- new net +VBAT_B: C26.1, C27.1, R40.1, R41.1, R42.1, U10.5 (VIN)
Changed lines of the file:
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@@
     (pin "1")
   )
-  (symbol (lib_id "RCAS_Power_Symbols:+VBAT_Enabled") (at 147.32 133.35 0) (unit 1)
-    (in_bom yes) (on_board yes)
-    (property "Reference" "#PWR066" (id 0) (at 147.32 137.16 0)
+  (symbol (lib_id "RCAS_Power_Symbols:+VBAT_B") (at 147.32 133.35 0) (unit 1)
+    (in_bom yes) (on_board yes) (fields_autoplaced)
+    (property "Reference" "#PWR?" (id 0) (at 147.32 137.16 0)
       (effects (font (size 1.27 1.27)) hide)
     )
-    (property "Value" "+VBAT_Enabled" (id 1) (at 147.701 128.9558 0))
+    (property "Value" "+VBAT_B" (id 1) (at 147.32 129.7742 0))
     (property "Footprint" "" (id 2) (at 147.32 133.35 0)
       (effects (font (size 1.27 1.27)) hide)
@@
     (pin "1")
   )
-  (symbol (lib_id "RCAS_Power_Symbols:+VBAT_Enabled") (at 229.87 58.42 0) (unit 1)
-    (in_bom yes) (on_board yes)
-    (property "Reference" "#PWR068" (id 0) (at 229.87 62.23 0)
+  (symbol (lib_id "RCAS_Power_Symbols:+VBAT_B") (at 229.87 58.42 0) (unit 1)
+    (in_bom yes) (on_board yes) (fields_autoplaced)
+    (property "Reference" "#PWR?" (id 0) (at 229.87 62.23 0)
       (effects (font (size 1.27 1.27)) hide)
     )
-    (property "Value" "+VBAT_Enabled" (id 1) (at 230.251 54.0258 0))
+    (property "Value" "+VBAT_B" (id 1) (at 229.87 54.8442 0))
     (property "Footprint" "" (id 2) (at 229.87 58.42 0)
       (effects (font (size 1.27 1.27)) hide)
