File: 2022/LocoMainBoard/Motor Control Interface.kicad_sch (KiCad schematic)
At the start: 37 parts, among them J1 D-Sub 9 Male, J2 Min-Fit Jr 2x08, Q1 2N7002, Q2 2N7002, Q3 FQD11P06TM, Q4 FQD11P06TM, Q5 2N7002, Q6 2N7002, Q7 2N7002, U1 MCP4716

Commit message: Full Rework of PCB --> basically V2
Connections:
- net +VBAT renamed +VBAT_B
Changed lines of the file:
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@@
     (pin "1")
   )
-  (symbol (lib_id "RCAS_Power_Symbols:+VBAT_Enabled") (at 72.39 46.99 0) (unit 1)
-    (in_bom yes) (on_board yes)
-    (property "Reference" "#PWR01" (id 0) (at 72.39 50.8 0)
+  (symbol (lib_id "RCAS_Power_Symbols:+VBAT_B") (at 72.39 46.99 0) (unit 1)
+    (in_bom yes) (on_board yes) (fields_autoplaced)
+    (property "Reference" "#PWR?" (id 0) (at 72.39 50.8 0)
       (effects (font (size 1.27 1.27)) hide)
     )
-    (property "Value" "+VBAT_Enabled" (id 1) (at 72.771 42.5958 0))
+    (property "Value" "+VBAT_B" (id 1) (at 72.39 43.4142 0))
     (property "Footprint" "" (id 2) (at 72.39 46.99 0)
       (effects (font (size 1.27 1.27)) hide)
