File: 2022/LocoMainBoard/Power & Interlocks.kicad_sch (KiCad schematic)
At the start: 57 parts, among them J14 Mini-Fit Jr 2x01, J15 Ethernet, J16 Ethernet, J17 Mini-Fit Jr 2x01, J18 Mini-Fit Jr 2x01, J20 Mini-Fit Jr 2x01, J23 Mini-Fit Jr 2x01, J32 Mini-Fit Jr 2x01, K1 FINDER-36.11, K2 FINDER-36.11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

Commit message: Full Rework of PCB --> basically V2
Connections:
- net +VBAT: no longer K3.11
- new net +VBAT_B: K3.11
Changed lines of the file:
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@@
+    (stroke (width 0) (type default) (color 0 0 0 0))
+  )
+  (wire (pts (xy 175.26 31.75) (xy 195.58 31.75))
     (stroke (width 0) (type default) (color 0 0 0 0))
   )
@@
   )
   (wire (pts (xy 36.83 191.77) (xy 36.83 194.31))
-    (stroke (width 0) (type default) (color 0 0 0 0))
-  )
-  (wire (pts (xy 175.26 31.75) (xy 195.58 31.75))
     (stroke (width 0) (type default) (color 0 0 0 0))
   )
@@
     (pin "1")
   )
-  (symbol (lib_id "RCAS_Power_Symbols:+VBAT_Enabled") (at 195.58 31.75 0) (unit 1)
-    (in_bom yes) (on_board yes)
-    (property "Reference" "#PWR0177" (id 0) (at 195.58 35.56 0)
-      (effects (font (size 1.27 1.27)) hide)
-    )
-    (property "Value" "+VBAT_Enabled" (id 1) (at 195.961 27.3558 0))
-    (property "Footprint" "" (id 2) (at 195.58 31.75 0)
-      (effects (font (size 1.27 1.27)) hide)
-    )
-    (property "Datasheet" "" (id 3) (at 195.58 31.75 0)
-      (effects (font (size 1.27 1.27)) hide)
-    )
-    (pin "1")
-  )
   (symbol (lib_id "RCAS_Power_Symbols:+VBAT") (at 151.13 29.21 0) (unit 1)
     (in_bom yes) (on_board yes)
@@
     (pin "2")
   )
+  (symbol (lib_id "RCAS_Power_Symbols:+VBAT_B") (at 195.58 31.75 0) (unit 1)
+    (in_bom yes) (on_board yes) (fields_autoplaced)
+    (property "Reference" "#PWR?" (id 0) (at 195.58 35.56 0)
+      (effects (font (size 1.27 1.27)) hide)
+    )
+    (property "Value" "+VBAT_B" (id 1) (at 195.58 28.1742 0))
+    (property "Footprint" "" (id 2) (at 195.58 31.75 0)
+      (effects (font (size 1.27 1.27)) hide)
+    )
+    (property "Datasheet" "" (id 3) (at 195.58 31.75 0)
+      (effects (font (size 1.27 1.27)) hide)
+    )
+    (pin "1")
+  )
 )
