File: 2022/LocoMainBoard/Processor.kicad_sch (KiCad schematic)
At the start: 55 parts, among them J19 Mini-Fit Jr 2x03, J21 Mini-Fit Jr 2x02, J22 Mini-Fit Jr 2x02, J24 Mini-Fit Jr 2x01, J25 Mini-Fit Jr 2x01, J26 Mini-Fit Jr 2x02, J27 Mini-Fit Jr 2x02, Q16 Q_NMOS_SSSGD, Q17 Q_NMOS_SSSGD, Q18 Q_NMOS_SSSGD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

Commit message: Full Rework of PCB --> basically V2
Parts:
- U16: footprint Module:ST_Morpho_Connector_144_STLink -> RCAS_Nucleo_F103RB:ST_NUCLEO-F103RB
Changed lines of the file:
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@@
     (property "Reference" "U16" (id 0) (at 308.737 86.8426 0))
     (property "Value" "NUCLEO64-F103RB" (id 1) (at 308.737 89.154 0))
-    (property "Footprint" "Module:ST_Morpho_Connector_144_STLink" (id 2) (at 287.02 190.5 0)
+    (property "Footprint" "RCAS_Nucleo_F103RB:ST_NUCLEO-F103RB" (id 2) (at 287.02 190.5 0)
       (effects (font (size 1.27 1.27)) (justify left) hide)
     )
