File: 2022/Control Box/Control Box.kicad_pcb (KiCad board)
At the start: 4 copper layers, 139.7 x 106.7 mm, 180 parts, among them J102 RJ45, J301 PicoBlade_1x02, J302 PicoBlade_1x02, J303 PicoBlade_1x02, J401 Conn_02x05_Odd_Even, J402 Conn_01x06, J403 Conn_01x06, J404 Mini USB, J501 PicoBlade_1x02, J601 PicoBlade_1x02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

Commit message: trial
Other:
- net class Default removed
- net class DiffPair removed
