File: 2022/Control Box/Power & Interlocks.kicad_sch (KiCad schematic)
At the start: 35 parts, among them J601 PicoBlade_1x02, J602 PicoBlade_1x04, J603 Barrel Jack, Q601 FQD11P06TM, Q602 2N7002, Q603 2N7002, Q604 2N7002

Commit message: rewired pcb nee to sort diff pairs
Parts:
- removed R616: 0R, symbol RCAS_Passives:Resistor
- R601: value 47R -> 0R
Connections:
- net at R601.1: now also D603.1 (A), Q603.3 (D)
Other:
- note removed: "SWAP AROUND OR DELETE R601?"
Changed lines of the file:
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@@
-    (stroke (width 0) (type default) (color 0 0 0 0))
-  )
-  (wire (pts (xy 58.42 50.8) (xy 66.04 50.8))
     (stroke (width 0) (type default) (color 0 0 0 0))
   )
@@
     (stroke (width 0) (type default) (color 0 0 0 0))
   )
-  (wire (pts (xy 73.66 50.8) (xy 88.9 50.8))
+  (wire (pts (xy 58.42 50.8) (xy 88.9 50.8))
     (stroke (width 0) (type default) (color 0 0 0 0))
   )
@@
   )
   (text "To start of interlock loop in loco" (at 259.08 160.02 0)
-    (effects (font (size 0.762 0.762)) (justify left bottom))
-  )
-  (text "SWAP AROUND OR DELETE R601?\n" (at 52.07 40.64 0)
     (effects (font (size 0.762 0.762)) (justify left bottom))
   )
@@
     (in_bom yes) (on_board yes)
     (property "Reference" "R601" (id 0) (at 54.61 45.5422 90))
-    (property "Value" "47R" (id 1) (at 54.61 47.8536 90))
+    (property "Value" "0R" (id 1) (at 54.61 47.8536 90))
     (property "Footprint" "RCAS_Resistor_SMD:R_0603_1608Metric_Pad1.05x0.95mm_HandSolder" (id 2) (at 54.61 49.022 90)
       (effects (font (size 1.27 1.27)) hide)
@@
     (property "Label" "E-STOP MOUNT" (id 4) (at 133.35 143.51 0))
   )
-  (symbol (lib_id "RCAS_Passives:Resistor") (at 69.85 50.8 90) (unit 1)
-    (in_bom yes) (on_board yes) (fields_autoplaced)
-    (property "Reference" "R616" (id 0) (at 69.85 44.45 90))
-    (property "Value" "0R" (id 1) (at 69.85 46.99 90))
-    (property "Footprint" "" (id 2) (at 69.85 52.578 90)
-      (effects (font (size 1.27 1.27)) hide)
-    )
-    (property "Datasheet" "~" (id 3) (at 69.85 50.8 0)
-      (effects (font (size 1.27 1.27)) hide)
-    )
-    (pin "1")
-    (pin "2")
-  )
 )
