File: 2022/Control Box/Control Box.kicad_sch (KiCad schematic)
At the start: 9 parts, among them J102 RJ45

Commit message: Control Box Ordering
Connections:
- net GND: now also J102.7 (Pin_7); no longer J102.2 (Pin_2)
- net INTERLOCK_OUT: now also J102.2 (Pin_2); no longer J102.7 (Pin_7)
- net POWER_EN: now also J102.1 (Pin_1); no longer J102.8 (Pin_8)
- net at F101.1: now also J102.8 (Pin_8); no longer J102.1 (Pin_1)
Other:
- moved on the sheet: C101, J102
