File: 2022/Interlock/Interlock/Interlock.kicad_sch (KiCad schematic)
At the start: 8 parts

Commit message: Made changes to interlock pcb -jb
Parts:
- added J3: Conn_01x02, RCAS_Connector_Molex:Molex_Mini-Fit_Jr_5566-02A_2x01_P4.20mm_Vertical, symbol RCAS_Connectors_Generic:Conn_01x02
- D3: renamed from D?; footprint (none) -> RCAS_Diode_SMD:D_0201_0603Metric
- J1, J2: renamed from J?; footprint (none) -> RCAS_Connector_Molex:Molex_Mini-Fit_Jr_5566-02A_2x01_P4.20mm_Vertical
- R2, R3: renamed from R?; footprint (none) -> RCAS_Resistor_SMD:R_0201_0603Metric
- gave numbers to parts that had none: 3
Connections:
- net GND: now also D1.1 (K), D2.1 (K), D3.1 (K), J1.1 (Pin_1), J2.2 (Pin_2), U1.1 (ADJ)
- net at R2.2, R3.1: now also J3.1 (Pin_1)
- net +3V3: now reaches J1.2 (Pin_2), J2.1 (Pin_1), R3.2, U1.3 (VIN)
Changed lines of the file:
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@@
   (junction (at 153.67 100.33) (diameter 0) (color 0 0 0 0)
+  )
+  (junction (at 88.9 85.09) (diameter 0) (color 0 0 0 0)
+  )
+  (junction (at 88.9 87.63) (diameter 0) (color 0 0 0 0)
   )
   (junction (at 173.99 85.09) (diameter 0) (color 0 0 0 0)
@@
     (stroke (width 0) (type default) (color 0 0 0 0))
   )
-  (wire (pts (xy 83.82 87.63) (xy 96.52 87.63))
+  (wire (pts (xy 83.82 87.63) (xy 88.9 87.63))
     (stroke (width 0) (type default) (color 0 0 0 0))
   )
@@
     (stroke (width 0) (type default) (color 0 0 0 0))
   )
+  (wire (pts (xy 88.9 87.63) (xy 96.52 87.63))
+    (stroke (width 0) (type default) (color 0 0 0 0))
+  )
   (wire (pts (xy 96.52 87.63) (xy 170.18 87.63))
     (stroke (width 0) (type default) (color 0 0 0 0))
@@
     (stroke (width 0) (type default) (color 0 0 0 0))
   )
-  (wire (pts (xy 83.82 85.09) (xy 100.33 85.09))
+  (wire (pts (xy 83.82 85.09) (xy 88.9 85.09))
     (stroke (width 0) (type default) (color 0 0 0 0))
   )
@@
     (stroke (width 0) (type default) (color 0 0 0 0))
   )
+  (wire (pts (xy 88.9 87.63) (xy 88.9 92.71))
+    (stroke (width 0) (type default) (color 0 0 0 0))
+  )
   (wire (pts (xy 170.18 87.63) (xy 170.18 107.95))
     (stroke (width 0) (type default) (color 0 0 0 0))
@@
     (stroke (width 0) (type default) (color 0 0 0 0))
   )
+  (wire (pts (xy 88.9 85.09) (xy 100.33 85.09))
+    (stroke (width 0) (type default) (color 0 0 0 0))
+  )
   (wire (pts (xy 153.67 107.95) (xy 160.02 107.95))
     (stroke (width 0) (type default) (color 0 0 0 0))
@@
     (stroke (width 0) (type default) (color 0 0 0 0))
   )
+  (wire (pts (xy 88.9 81.28) (xy 88.9 85.09))
+    (stroke (width 0) (type default) (color 0 0 0 0))
+  )
   (wire (pts (xy 96.52 105.41) (xy 96.52 87.63))
     (stroke (width 0) (type default) (color 0 0 0 0))
@@
   (symbol (lib_id "RCAS_Passives:Resistor") (at 143.51 69.85 90) (unit 1)
     (in_bom yes) (on_board yes) (fields_autoplaced)
-    (property "Reference" "R?" (id 0) (at 143.51 63.5 90))
+    (property "Reference" "R2" (id 0) (at 143.51 63.5 90))
     (property "Value" "Resistor" (id 1) (at 143.51 66.04 90))
-    (property "Footprint" "" (id 2) (at 143.51 71.628 90)
+    (property "Footprint" "RCAS_Resistor_SMD:R_0201_0603Metric" (id 2) (at 143.51 71.628 90)
       (effects (font (size 1.27 1.27)) hide)
     )
@@
   (symbol (lib_id "RCAS_Connectors_Generic:Conn_01x02") (at 78.74 87.63 180) (unit 1)
     (in_bom yes) (on_board yes) (fields_autoplaced)
-    (property "Reference" "J?" (id 0) (at 78.74 78.74 0))
+    (property "Reference" "J1" (id 0) (at 78.74 78.74 0))
     (property "Value" "Conn_01x02" (id 1) (at 78.74 81.28 0))
-    (property "Footprint" "" (id 2) (at 78.74 87.63 0)
+    (property "Footprint" "RCAS_Connector_Molex:Molex_Mini-Fit_Jr_5566-02A_2x01_P4.20mm_Vertical" (id 2) (at 78.74 87.63 0)
       (effects (font (size 1.27 1.27)) hide)
     )
@@
   (symbol (lib_id "RCAS_Connectors_Generic:Conn_01x02") (at 184.15 85.09 0) (unit 1)
     (in_bom yes) (on_board yes)
-    (property "Reference" "J?" (id 0) (at 186.69 85.0899 0)
+    (property "Reference" "J2" (id 0) (at 186.69 85.0899 0)
       (effects (font (size 1.27 1.27)) (justify left))
     )
@@
       (effects (font (size 1.27 1.27)) (justify left))
     )
-    (property "Footprint" "" (id 2) (at 184.15 85.09 0)
+    (property "Footprint" "RCAS_Connector_Molex:Molex_Mini-Fit_Jr_5566-02A_2x01_P4.20mm_Vertical" (id 2) (at 184.15 85.09 0)
       (effects (font (size 1.27 1.27)) hide)
     )
@@
   (symbol (lib_id "RCAS_LEDs:LED") (at 147.32 104.14 90) (unit 1)
     (in_bom yes) (on_board yes) (fields_autoplaced)
-    (property "Reference" "D?" (id 0) (at 151.13 104.4574 90)
+    (property "Reference" "D1" (id 0) (at 151.13 104.4574 90)
       (effects (font (size 1.27 1.27)) (justify right))
     )
@@
     (pin "2")
   )
+  (symbol (lib_id "RCAS_Power_Symbols:GND") (at 88.9 92.71 0) (unit 1)
+    (in_bom yes) (on_board yes) (fields_autoplaced)
+    (property "Reference" "#PWR?" (id 0) (at 88.9 99.06 0)
+      (effects (font (size 1.27 1.27)) hide)
+    )
+    (property "Value" "GND" (id 1) (at 88.9 97.79 0))
+    (property "Footprint" "" (id 2) (at 88.9 92.71 0)
+      (effects (font (size 1.27 1.27)) hide)
+    )
+    (property "Datasheet" "" (id 3) (at 88.9 92.71 0)
+      (effects (font (size 1.27 1.27)) hide)
+    )
+    (pin "1")
+  )
   (symbol (lib_id "RCAS_Passives:Resistor") (at 154.94 69.85 90) (unit 1)
     (in_bom yes) (on_board yes) (fields_autoplaced)
-    (property "Reference" "R?" (id 0) (at 154.94 63.5 90))
+    (property "Reference" "R3" (id 0) (at 154.94 63.5 90))
     (property "Value" "Resistor" (id 1) (at 154.94 66.04 90))
-    (property "Footprint" "" (id 2) (at 154.94 71.628 90)
+    (property "Footprint" "RCAS_Resistor_SMD:R_0201_0603Metric" (id 2) (at 154.94 71.628 90)
       (effects (font (size 1.27 1.27)) hide)
     )
@@
   (symbol (lib_id "RCAS_LM350AT_NOPB:LM350AT{slash}NOPB") (at 123.19 102.87 0) (unit 1)
     (in_bom yes) (on_board yes) (fields_autoplaced)
-    (property "Reference" "U?" (id 0) (at 123.19 92.71 0))
+    (property "Reference" "U1" (id 0) (at 123.19 92.71 0))
     (property "Value" "LM350AT/NOPB" (id 1) (at 123.19 95.25 0))
     (property "Footprint" "TO254P1054X470X1955-3" (id 2) (at 123.19 102.87 0)
@@
     (pin "3")
   )
+  (symbol (lib_id "RCAS_Connectors_Generic:Conn_01x02") (at 175.26 59.69 0) (unit 1)
+    (in_bom yes) (on_board yes) (fields_autoplaced)
+    (property "Reference" "J3" (id 0) (at 177.8 59.6899 0)
+      (effects (font (size 1.27 1.27)) (justify left))
+    )
+    (property "Value" "Conn_01x02" (id 1) (at 177.8 62.2299 0)
+      (effects (font (size 1.27 1.27)) (justify left))
+    )
+    (property "Footprint" "RCAS_Connector_Molex:Molex_Mini-Fit_Jr_5566-02A_2x01_P4.20mm_Vertical" (id 2) (at 175.26 59.69 0)
+      (effects (font (size 1.27 1.27)) hide)
+    )
+    (property "Datasheet" "~" (id 3) (at 175.26 59.69 0)
+      (effects (font (size 1.27 1.27)) hide)
+    )
+    (pin "1")
+    (pin "2")
+  )
   (symbol (lib_id "RCAS_LEDs:LED") (at 160.02 104.14 90) (unit 1)
     (in_bom yes) (on_board yes) (fields_autoplaced)
-    (property "Reference" "D?" (id 0) (at 163.83 104.4574 90)
+    (property "Reference" "D3" (id 0) (at 163.83 104.4574 90)
       (effects (font (size 1.27 1.27)) (justify right))
     )
@@
       (effects (font (size 1.27 1.27)) (justify right))
     )
-    (property "Footprint" "" (id 2) (at 160.02 104.14 0)
+    (property "Footprint" "RCAS_Diode_SMD:D_0201_0603Metric" (id 2) (at 160.02 104.14 0)
       (effects (font (size 1.27 1.27)) hide)
     )
@@
     (pin "2")
   )
+  (symbol (lib_id "RCAS_Power_Symbols:+3V3") (at 88.9 81.28 0) (unit 1)
+    (in_bom yes) (on_board yes) (fields_autoplaced)
+    (property "Reference" "#PWR?" (id 0) (at 88.9 85.09 0)
+      (effects (font (size 1.27 1.27)) hide)
+    )
+    (property "Value" "+3V3" (id 1) (at 88.9 76.2 0))
+    (property "Footprint" "" (id 2) (at 88.9 81.28 0)
+      (effects (font (size 1.27 1.27)) hide)
+    )
+    (property "Datasheet" "" (id 3) (at 88.9 81.28 0)
+      (effects (font (size 1.27 1.27)) hide)
+    )
+    (pin "1")
+  )
   (symbol (lib_id "RCAS_LEDs:LED") (at 153.67 104.14 90) (unit 1)
     (in_bom yes) (on_board yes) (fields_autoplaced)
-    (property "Reference" "D?" (id 0) (at 157.48 104.4574 90)
+    (property "Reference" "D2" (id 0) (at 157.48 104.4574 90)
       (effects (font (size 1.27 1.27)) (justify right))
     )
@@
   )
   (symbol_instances
+    (path "/7349e54d-5dc8-40f7-98bc-152460f817df"
+      (reference "#PWR?") (unit 1) (value "GND") (footprint "")
+    )
+    (path "/cc40f5e6-09f9-43de-9373-8a7e52fb4c51"
+      (reference "#PWR?") (unit 1) (value "+3V3") (footprint "")
+    )
     (path "/e05a8fcc-3be1-4a7d-af80-5bd92f3bda04"
       (reference "#PWR?") (unit 1) (value "GND") (footprint "")
     )
     (path "/6a91ecf2-b999-4311-946f-c179b050b8c4"
-      (reference "D?") (unit 1) (value "LED") (footprint "")
+      (reference "D1") (unit 1) (value "LED") (footprint "")
+    )
+    (path "/d0ec0fe0-0ec3-4983-b901-4476725de6f4"
+      (reference "D2") (unit 1) (value "LED") (footprint "")
     )
     (path "/91e22fa1-f43e-4304-95e3-f8dfde94ddee"
-      (reference "D?") (unit 1) (value "LED") (footprint "")
-    )
-    (path "/d0ec0fe0-0ec3-4983-b901-4476725de6f4"
-      (reference "D?") (unit 1) (value "LED") (footprint "")
+      (reference "D3") (unit 1) (value "LED") (footprint "RCAS_Diode_SMD:D_0201_0603Metric")
     )
     (path "/1ff96fa7-9cc1-42db-907d-2e235000d1c3"
-      (reference "J?") (unit 1) (value "Conn_01x02") (footprint "")
+      (reference "J1") (unit 1) (value "Conn_01x02") (footprint "RCAS_Connector_Molex:Molex_Mini-Fit_Jr_5566-02A_2x01_P4.20mm_Vertical")
     )
     (path "/4afef8e7-cd32-47fc-8df0-fd0d702eec77"
-      (reference "J?") (unit 1) (value "Conn_01x02") (footprint "")
+      (reference "J2") (unit 1) (value "Conn_01x02") (footprint "RCAS_Connector_Molex:Molex_Mini-Fit_Jr_5566-02A_2x01_P4.20mm_Vertical")
+    )
+    (path "/91d74263-4204-417f-ba51-473f10770e00"
+      (reference "J3") (unit 1) (value "Conn_01x02") (footprint "RCAS_Connector_Molex:Molex_Mini-Fit_Jr_5566-02A_2x01_P4.20mm_Vertical")
     )
     (path "/1a2f2da4-3b90-4f8b-ab60-4fd986aa620b"
-      (reference "R?") (unit 1) (value "Resistor") (footprint "")
+      (reference "R2") (unit 1) (value "Resistor") (footprint "RCAS_Resistor_SMD:R_0201_0603Metric")
     )
     (path "/81f563ab-6504-4912-b26c-c449605c6efe"
-      (reference "R?") (unit 1) (value "Resistor") (footprint "")
+      (reference "R3") (unit 1) (value "Resistor") (footprint "RCAS_Resistor_SMD:R_0201_0603Metric")
     )
     (path "/8e8f4cf7-7eea-48ca-ae3c-7f5752270791"
-      (reference "U?") (unit 1) (value "LM350AT/NOPB") (footprint "TO254P1054X470X1955-3")
-    )
-  )
+      (reference "U1") (unit 1) (value "LM350AT/NOPB") (footprint "TO254P1054X470X1955-3")
+    )
+  )
